File: electronics/klipper-switch/switches.kicad_sch (KiCad schematic)
At the start: 0 parts

Commit message: schematic naming and pico symbol update
Other:
- title: (none) -> klipper-switch, switches
Changed lines of the file:
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@@
 	(generator_version "8.0")
 	(paper "A4")
+	(title_block
+		(title "klipper-switch, switches")
+	)
 )
