File: electronics/klipper-switch/connectors.kicad_sch (KiCad schematic)
At the start: 0 parts

Commit message: Added BV1 Footprint properly and fixed my libraries
Parts:
- added J1: Conn_01x04_Socket, symbol Connector:Conn_01x04_Socket
- added J2: Conn_02x03_Odd_Even, symbol Connector_Generic:Conn_02x03_Odd_Even
Connections:
- new net: J1.2 (Pin_2), J2.1 (Pin_1), J2.3 (Pin_3), J2.5 (Pin_5)
