File: electronics/klipper-switch/LEDs.kicad_sch (KiCad schematic)
At the start: 17 parts, among them Q1 RK7002BMT116, Q2 RK7002BMT116, Q3 RK7002BMT116

Commit message: completed rough schematic
Parts:
- added D10, D11, D12, D13, D14, D15, D16, D17, D18, D19, D8, D9: 151031SS06000, LED_THT:LED_D3.0mm, symbol klipper-switch:151031SS06000
- added Q10, Q11, Q12, Q13, Q14, Q15, Q4, Q5, Q6, Q7, Q8, Q9: RK7002BMT116, klipper-switch:RK7002BMT116, symbol klipper-switch:RK7002BMT116
- added R40, R42, R43, R45, R46, R48, R49, R51, R52, R53, R56, R57, R58, R59, R62, R63, R64, R65, R68, R69, R70, R71, R74, R75: 100R, Resistor_SMD:R_1206_3216Metric, symbol klipper-switch:RC1206FR-7W100RL_1
- added R41, R44, R47, R50, R54, R55, R60, R61, R66, R67, R72, R73: 10K, Resistor_SMD:R_1206_3216Metric, symbol klipper-switch:RC1206FR-7W100RL_1
Connections:
- net +5V: now also R40.1, R45.1, R48.1, R51.1, R56.1, R57.1, R62.1, R63.1, R68.1, R69.1, R74.1, R75.1
- net GND: now also Q10.1 (S), Q11.1 (S), Q12.1 (S), Q13.1 (S), Q14.1 (S), Q15.1 (S), Q4.1 (S), Q5.1 (S), Q6.1 (S), Q7.1 (S), Q8.1 (S), Q9.1 (S), R41.2, R44.2, R47.2, R50.2, R54.2, R55.2, R60.2, R61.2, R66.2, R67.2, R72.2, R73.2
- new net: Q15.2 (G), R71.2, R73.1
- new net: D19.1 (K), Q15.3 (D)
- new net: Q14.2 (G), R70.2, R72.1
- new net: D18.1 (K), Q14.3 (D)
- new net: Q13.2 (G), R65.2, R67.1
- new net: D19.2 (A), R75.2
- new net: Q5.2 (G), R43.2, R44.1
- new net: D9.1 (K), Q5.3 (D)
- new net: D9.2 (A), R45.2
- new net: Q9.2 (G), R53.2, R55.1
- new net: D11.2 (A), R51.2
- new net: D13.1 (K), Q9.3 (D)
- new net: D14.2 (A), R62.2
- new net: D13.2 (A), R57.2
- new net: Q8.2 (G), R52.2, R54.1
- new net: Q7.2 (G), R49.2, R50.1
- new net: Q4.2 (G), R41.1, R42.2
- new net: D8.1 (K), Q4.3 (D)
- new net: D12.2 (A), R56.2
- new net: Q11.2 (G), R59.2, R61.1
- new net: D10.1 (K), Q6.3 (D)
- new net: D10.2 (A), R48.2
- new net: D15.1 (K), Q11.3 (D)
- new net: D15.2 (A), R63.2
- new net: Q12.2 (G), R64.2, R66.1
- new net: Q6.2 (G), R46.2, R47.1
- new net: D16.2 (A), R68.2
- new net: D16.1 (K), Q12.3 (D)
- new net: Q10.2 (G), R58.2, R60.1
- new net: D11.1 (K), Q7.3 (D)
- new net: D12.1 (K), Q8.3 (D)
- new net: D8.2 (A), R40.2
- new net: D17.2 (A), R69.2
- new net: D14.1 (K), Q10.3 (D)
- new net: D17.1 (K), Q13.3 (D)
- new net: D18.2 (A), R74.2
- new net LED_CH_A: R42.1
- new net LED_CH_B: R43.1
- new net LED_CH_C: R46.1
- new net LED_CH_D: R49.1
- new net LED_CH_E: R52.1
- new net LED_CH_F: R58.1
- new net LED_CH_G: R53.1
- new net LED_CH_H: R59.1
- new net LED_CH_I: R64.1
- new net LED_CH_J: R70.1
- new net LED_CH_K: R65.1
- new net LED_CH_L: R71.1
Other:
- moved on the sheet: D1, D2, D3, D4, D5, D6, D7, Q1, Q2, Q3, R1, R2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
