File: electronics/klipper-switch/opto-isolators.kicad_sch (KiCad schematic)
At the start: 0 parts

Commit message: schematic naming and pico symbol update
Other:
- title: (none) -> klipper-switch, opto-isolators
Changed lines of the file:
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@@
 	(generator_version "8.0")
 	(paper "A4")
+	(title_block
+		(title "klipper-switch, opto-isolators")
+		(rev "V 1.0")
+	)
 )

Commit message: completed rough schematic
Parts:
- added R24, R26, R28, R29, R32, R33, R36, R37, R84, R85, R88, R89: 2.4K, Resistor_SMD:R_1206_3216Metric, symbol klipper-switch:RC1206FR-7W100RL_1
- added R25, R27, R30, R31, R34, R35, R38, R39, R86, R87, R90, R91: 100K, Resistor_SMD:R_1206_3216Metric, symbol klipper-switch:RC1206FR-07100KL
- added U10, U11, U12, U13, U14, U15, U16, U17, U22, U23, U24, U25: LTV-356T, Package_SO:SO-4_4.4x3.6mm_P2.54mm, symbol klipper-switch:LTV-356T
Connections:
- new net: R28.2, U12.1
- new net: R29.2, U13.1
- new net: R24.2, U10.1
- new net: R88.2, U24.1
- new net: R36.2, U16.1
- new net: R32.2, U14.1
- new net: R89.2, U25.1
- new net: R85.2, U23.1
- new net: R84.2, U22.1
- new net: R37.2, U17.1
- new net: R26.2, U11.1
- new net: R33.2, U15.1
- new net +3.3V: R25.2, R27.2, R30.2, R31.2, R34.2, R35.2, R38.2, R39.2, R86.2, R87.2, R90.2, R91.2
- new net GND: U10.2, U10.3, U11.2, U11.3, U12.2, U12.3, U13.2, U13.3, U14.2, U14.3, U15.2, U15.3, U16.2, U16.3, U17.2, U17.3, U22.2, U22.3, U23.2, U23.3, U24.2, U24.3, U25.2, U25.3
- new net IN_CH_A: R24.1
- new net IN_CH_B: R28.1
- new net IN_CH_C: R26.1
- new net IN_CH_D: R29.1
- new net IN_CH_E: R32.1
- new net IN_CH_F: R36.1
- new net IN_CH_G: R33.1
- new net IN_CH_H: R37.1
- new net IN_CH_I: R84.1
- new net IN_CH_J: R88.1
- new net IN_CH_K: R85.1
- new net IN_CH_L: R89.1
- new net OUT_CH_A: R25.1, U10.4
- new net OUT_CH_B: R30.1, U12.4
- new net OUT_CH_C: R27.1, U11.4
- new net OUT_CH_D: R31.1, U13.4
- new net OUT_CH_E: R34.1, U14.4
- new net OUT_CH_F: R38.1, U16.4
- new net OUT_CH_G: R35.1, U15.4
- new net OUT_CH_H: R39.1, U17.4
- new net OUT_CH_I: R86.1, U22.4
- new net OUT_CH_J: R90.1, U24.4
- new net OUT_CH_K: R87.1, U23.4
- new net OUT_CH_L: R91.1, U25.4
